File: docs/smbus_programmer.kicad_sch (KiCad schematic)
At the start: 5 parts, among them J1 4SU0016, U1 ESP32-WROOM-32D, U2 TCA9548A

Commit message: programmer schematics update
Parts:
- added R3, R4: 3.3k, Resistor_SMD:R_0805_2012Metric, symbol R
Connections:
- net +3V3: now also R3.1, R4.1
- net GND: now also J1.GND
- new net RL78_RESET: J1.8 (RESET), U1.27 (IO16_RESET)
- new net RXD0: J1.5 (RXD0), U1.10 (IO25_RXD0)
- new net TOOL0: J1.7 (TOOL0), R3.2, U1.28 (IO17_TOOL0)
- new net TXD0: J1.6 (TXD0), R4.2, U1.11 (IO26_TXD0)
Other:
- note added: "Channel 3 only. SD3 (TCA9548A pin 10) goes to 4SU0016 pin 128 SDA. SC3 (pin 11) goes to pin 127 SCL."
- note added: "ESP32-WROOM-32D. 3.3 V is the module regulator, separate from the pack. Pack positive is not connected."
- note added: "GND symbols are one net: ESP32 ground and 4SU0016 ground."
- note added: "GPIO16 (module pin 27) drives pin 8 RESET, PCB plate 28, direct, no pull-up."
- note added: "GPIO17 (module pin 28) drives pin 7 TOOL0, PCB plate 29. R3 is 3.3 kOhm from TOOL0 to 3.3 V."
- note added: "GPIO26 (module pin 11) reads pin 6 TxD0. R4 is 3.3 kOhm from pin 6 to 3.3 V."
- note added: "Programming UART, 115200 8N2. GPIO25 (module pin 10) drives RAJ240045 pin 5 RxD0, direct."
- note added: "R1 and R2 are 3.3 kOhm from 3.3 V to SD3 and SC3."
- note added: "RAJ240045"
- note added: "plate 28"
- note added: "plate 29"
- note removed: "4SU0016 ground"
- note removed: "Channel 3 only. SD3 (TCA9548A pin 10) goes to 4SU0016 pin 128, SDA. SC3 (pin 11) goes to 4SU0016 pin 127, SCL."
- note removed: "ESP32-WROOM-32D board. 3.3 V comes from the ESP32 regulator, a separate supply from the pack. Pack positive is not connected."
- note removed: "R1 and R2 are 3.3 kOhm from the ESP32 3.3 V rail to SD3 and SC3. Channels 0-2 and 4-7 are not part of this adapter."
- note removed: "The GND symbols are one net: ESP32 ground and 4SU0016 ground."
